File: STM32 MCU.kicad_sch (KiCad schematic)
At the start: 32 parts, among them J4 Conn_01x04_Pin, J5 Conn_01x02_Pin, SW2 SW_Push, SW5 SW_Push, U3 STM32G474RETx, Y1 16MHz

Commit message: got rid of pins on stm32
Connections:
- net SPI_CS_ESP: no longer names the net of U3.22 (PC4)
Changed lines of the file:
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@@
-	(wire
-		(pts
-			(xy 31.75 69.85) (xy 52.07 69.85)
-		)
-		(stroke
-			(width 0)
-			(type default)
-			(color 221 133 0 1)
-		)
-	)
 	(wire
 		(pts
@@
 		)
 	)
-	(hierarchical_label "SPI_CS_ESP"
-		(shape input)
-		(at 31.75 69.85 180)
-		(effects
-			(font
-				(size 1.27 1.27)
-			)
-			(justify right)
-		)
-	)
